File: PCB/MkII/CCCCPPPS_MkII.kicad_pcb (KiCad board)
At the start: 2 copper layers, 30 parts, among them J1 PROG_HEADER, J2 USB_C, J3 CONN_OUT, J4 CONN_IN, Q1 AO3400A, U1 AMS1117-3.3, U2 CH32V003AxMx

Commit message: PCB Near final
Parts:
- removed U1: AMS1117-3.3, Package_TO_SOT_SMD:SOT-223-3_TabPin2
- added U3: AP2112K-3.3, Package_TO_SOT_SMD:SOT-23-5, F.Cu at (130.7, 143.3)
- moved R1 123.2 mm to (129.1, 151.2)
- moved R2 117.8 mm to (128.1, 155.2), turned to -90 degrees
- moved J1 116.7 mm to (135.5, 147.0), turned to -90 degrees
- moved J2 115.5 mm to (121.1, 152.5)
- moved C2 115.4 mm to (134.1, 143.3), turned to -90 degrees
- moved R7 113.5 mm to (142.9, 154.9), turned to -90 degrees
- moved R3 110.6 mm to (130.1, 155.2), turned to -90 degrees
- moved U2 108.9 mm to (136.6, 152.9), turned to 90 degrees
- moved R8 108.0 mm to (142.9, 150.9), turned to -90 degrees
- moved C1 107.6 mm to (127.2, 143.3), turned to -90 degrees
- moved C3 100.5 mm to (136.2, 143.3)
- moved J4 42.4 mm to (120.9, 141.1)
- moved C8 13.7 mm to (141.1, 143.9), turned to -90 degrees
- moved R9 7.83 mm to (162.7, 141.1), turned to 180 degrees
- moved J3 5.89 mm to (171.1, 144.6)
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Connections:
- net /USB_DM renamed /USB_DN
- net Net-(D1-A) renamed /L_OUT
- net Net-(Q1-D) renamed /L_IN
Routing:
- net VBUS_OUT_NEG: track 0.00 -> 40.3 mm, vias 0 -> 1
- net /VOUT_FB: track 1.93 -> 32.6 mm, vias 1 -> 2
- net /PSU_PWM: track 2.09 -> 18.9 mm, vias 0 -> 2
- net GND: track 23.2 -> 11.5 mm, vias 18 -> 28
- net /SWIO: track 2.53 -> 13.5 mm, vias 0 -> 1
- net VBUS_3V3: track 6.28 -> 15.1 mm, vias 1 -> 0
- net /USB_DP: track 20.9 -> 13.2 mm
- net /USB_DN: track 21.4 -> 14.1 mm
- net VBUS_5V_USB: track 2.56 -> 7.77 mm, vias 6 -> 10
- net Net-(J2-CC1): track 6.98 -> 3.27 mm
- net Net-(J2-CC2): track 6.49 -> 3.27 mm
- net /USB_DPU: track 2.58 -> 4.55 mm
- added copper zone on F.Cu, net /L_IN
- added copper zone on F.Cu, net /L_OUT
- added copper zone on B.Cu, net GND
- added copper zone on F.Cu, net GND
- added copper zone on B.Cu, net VBUS_5V_USB
- added copper zone on F.Cu, net VBUS_5V_USB
- added copper zone on F.Cu, net VBUS_OUT_NEG
- added copper zone on F.Cu, net VBUS_OUT_POS

Commit message: Full Refactor
Parts:
- removed C3: 100nF, Capacitor_SMD:C_0805_2012Metric
- added JP1: JMP_USB_VIN, Jumper:SolderJumper-2_P1.3mm_Open_RoundedPad1.0x1.5mm, B.Cu at (25.4, 33.5)
- J1: footprint Connector_PinSocket_2.54mm:PinSocket_1x03_P2.54mm_Vertical -> Connector_PinHeader_2.54mm:PinHeader_1x03_P2.54mm_Vertical
- TP1, TP3, TP4: footprint TestPoint:TestPoint_Pad_D3.0mm -> TestPoint:TestPoint_Pad_D1.5mm; moved to B.Cu
- TP2: value 5V -> VIN; footprint TestPoint:TestPoint_Pad_D3.0mm -> TestPoint:TestPoint_Pad_D1.5mm; moved to B.Cu
- moved TP2 196.9 mm to (28.4, 28.6), turned to 180 degrees
- moved TP4 192.3 mm to (37.5, 28.6), turned to 180 degrees
- moved TP3 188.8 mm to (33.0, 28.6), turned to 180 degrees
- moved TP1 166.6 mm to (65.2, 39.1), turned to 180 degrees
- moved J3 153.2 mm to (70.2, 29.2), turned to -90 degrees
- moved C4 150.6 mm to (50.9, 42.4)
- moved C5 150.6 mm to (63.1, 43.0)
- moved C7 150.6 mm to (61.6, 36.4)
- moved C8 150.6 mm to (40.1, 32.1)
- moved D1 150.6 mm to (56.2, 43.1)
- moved J1 150.6 mm to (34.6, 35.2)
- moved L1 150.6 mm to (50.8, 34.4)
- moved Q1 150.6 mm to (47.1, 43.1)
- moved R3 150.6 mm to (29.2, 43.4)
- moved R4 150.6 mm to (44.1, 43.1)
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Connections:
- C1 pad 1: VBUS_5V_USB -> VBUS_VIN
- C8 pad 1: VBUS_5V_USB -> VBUS_VIN
- J2 pad A4: VBUS_5V_USB -> /VBUS_USB
- J2 pad A9: VBUS_5V_USB -> /VBUS_USB
- J2 pad B4: VBUS_5V_USB -> /VBUS_USB
- J2 pad B9: VBUS_5V_USB -> /VBUS_USB
- J3 pad 1: VBUS_OUT_POS -> VBUS_OUT_NEG
- J3 pad 2: VBUS_OUT_NEG -> VBUS_OUT_POS
- J4 pad 1: VBUS_5V_USB -> GND
- J4 pad 2: GND -> VBUS_VIN
- L1 pad 2: VBUS_5V_USB -> VBUS_VIN
- TP2 pad 1: VBUS_5V_USB -> VBUS_VIN
- U3 pad 1: VBUS_5V_USB -> VBUS_VIN
- U3 pad 3: VBUS_5V_USB -> VBUS_VIN
Routing:
- net VBUS_5V_USB: track 7.77 -> 0.00 mm, vias 10 -> 0
- net VBUS_VIN: track 0.00 -> 7.27 mm, vias 0 -> 5
- net /PSU_PWM: track 18.9 -> 21.7 mm
- net /SWIO: track 13.5 -> 15.3 mm, vias 1 -> 0
- net VBUS_3V3: track 15.1 -> 13.8 mm, vias 0 -> 1
- net GND: track 11.5 -> 10.9 mm
- net VBUS_OUT_POS: vias 0 -> 1
- net /VBUS_USB: vias 0 -> 6
- added copper zone on B.Cu, net /VBUS_USB
- added copper zone on F.Cu, net /VBUS_USB
- added copper zone on B.Cu, net VBUS_VIN
- added copper zone on F.Cu, net VBUS_VIN
- removed copper zone on B.Cu, net VBUS_5V_USB
- removed copper zone on F.Cu, net VBUS_5V_USB
Other:
- board outline added: 58 x 20 mm
- board text added: "2024 MkII ADBeta Bogdan Ionescu"
- board text added: "JMP VIN USB"
- board text added: "VIN 6v MAX"
- board text added: "VOUT"
