File: PCB/MkII/CCCCPPPS_MkII.kicad_sch (KiCad schematic)
At the start: 23 parts, among them J1 USB_C, J2 PROG_HEADER, Q1 AO3400A, U1 CH32V003AxMx, U2 AMS1117-3.3

Commit message: MkII PCB Update
Parts:
- removed C4: 100uF, Capacitor_THT:CP_Radial_D6.3mm_P2.50mm, symbol Device:C_Polarized
- removed C5, C6: 10uF, Capacitor_SMD:C_0805_2012Metric_Pad1.18x1.45mm_HandSolder, symbol Device:C
- removed C7: 100uF 25V, Capacitor_THT:CP_Radial_D6.3mm_P2.50mm, symbol Device:C_Polarized
- removed D1: B2100-13-F, Diode_SMD:D_SMB_Handsoldering, symbol Device:D_Schottky
- added C4, C6: 10uF, Capacitor_SMD:C_0805_2012Metric, symbol Device:C_Small
- added C5: 100nF, Capacitor_SMD:C_0805_2012Metric, symbol Device:C_Small
- added C7, C8: 100uF, Capacitor_SMD:CP_Elec_6.3x5.2, symbol Device:C_Polarized_Small
- added D1: SS34, Diode_SMD:D_SMA, symbol Diode:SS34
- added J3: CONN_OUT, Custom_Footprints:PCB_Terminal_Block_2-P3.5, symbol Connector:Screw_Terminal_01x02
- added J4: CONN_IN, Custom_Footprints:PCB_Terminal_Block_2-P3.5, symbol Connector:Screw_Terminal_01x02
- added TP1: VOUT, TestPoint:TestPoint_Pad_D3.0mm, symbol Connector:TestPoint
- added TP2: 5V, TestPoint:TestPoint_Pad_D3.0mm, symbol Connector:TestPoint
- added TP3: 3V3, TestPoint:TestPoint_Pad_D3.0mm, symbol Connector:TestPoint
- added TP4: GND, TestPoint:TestPoint_Pad_D3.0mm, symbol Connector:TestPoint
- C1, C2: value 1uF -> 10uF; footprint Capacitor_SMD:C_0603_1608Metric -> Capacitor_SMD:C_0805_2012Metric
- C3: footprint Capacitor_SMD:C_0603_1608Metric -> Capacitor_SMD:C_0805_2012Metric
- R1, R2, R3: footprint Resistor_SMD:R_0603_1608Metric -> Resistor_SMD:R_0805_2012Metric
- R4: value 10k -> 10K; footprint Resistor_SMD:R_0603_1608Metric_Pad0.98x0.95mm_HandSolder -> Resistor_SMD:R_0805_2012Metric
- R5: renamed from R1; value 39k -> 39K; footprint Resistor_SMD:R_0603_1608Metric_Pad0.98x0.95mm_HandSolder -> Resistor_SMD:R_0805_2012Metric
- R6: renamed from R4; value 10k -> 10K; footprint Resistor_SMD:R_0603_1608Metric_Pad0.98x0.95mm_HandSolder -> Resistor_SMD:R_0805_2012Metric
- R7: renamed from R10; footprint Resistor_SMD:R_0603_1608Metric_Pad0.98x0.95mm_HandSolder -> Resistor_SMD:R_0805_2012Metric
- R8: renamed from R5; footprint Resistor_SMD:R_0603_1608Metric_Pad0.98x0.95mm_HandSolder -> Resistor_SMD:R_0805_2012Metric
- R9: value 333mR -> 330mR; footprint Resistor_SMD:R_1210_3225Metric_Pad1.30x2.65mm_HandSolder -> Resistor_SMD:R_2512_6332Metric_Pad1.40x3.35mm_HandSolder
- renumbered J2 to J1, J1 to J2, U2 to U1, U1 to U2
Connections:
- net VPP is gone; now on net VBUS_5V_USB: L1.2
- net GND: now also J1.2 (Pin_2), C5.2, C6.2, C7.2, C8.2, J4.2 (Pin_2), TP4.1; no longer J1.3 (Pin_3)
- net SWIO: now also J1.3 (Pin_3); no longer J1.2 (Pin_2)
- net VBUS_3V3: now also TP3.1
- net VBUS_5V_USB: now also C8.1, J4.1 (Pin_1), TP2.1
- net VBUS_OUT_NEG: now also J3.2 (Pin_2)
- net VBUS_OUT_POS: now also C5.1, C6.1, C7.1, D1.1 (K), J3.1 (Pin_1), TP1.1
- net at L1.3: now also C4.2, D1.2 (A)
- net at L1.4, Q1.3 (D): now also C4.1
- net PWM_OUT renamed PSU_PWM
- no-connect marks 2 -> 7
Other:
- note added: "Current Sense Amp"
- note added: "Output Connector"
- note added: "SEPIC Converter"
- moved on the sheet: C1, C2, C3, J1, J2, L1, Q1, R1, R2, R3, R4, R5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

Commit message: PCB Near final
Parts:
- removed U1: AMS1117-3.3, Package_TO_SOT_SMD:SOT-223-3_TabPin2, symbol Regulator_Linear:AMS1117-3.3
- added U3: AP2112K-3.3, Package_TO_SOT_SMD:SOT-23-5, symbol Regulator_Linear:AP2112K-3.3
Connections:
- net GND: now also U3.2 (GND)
- net VBUS_3V3: now also U3.5 (VOUT)
- net VBUS_5V_USB: now also U3.1 (VIN), U3.3 (EN)
- net L_OUT: now reaches C4.2, D1.2 (A), L1.3
- net L_IN: now reaches C4.1, L1.4, Q1.3 (D)
- net USB_DM renamed USB_DN
Other:
- moved on the sheet: C1, C2
Changed lines of the file:
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@@
 	)
 	(junction
+		(at 83.82 24.13)
+		(diameter 0)
+		(color 0 0 0 0)
+	)
+	(junction
 		(at 42.545 41.91)
 		(diameter 0)
@@
 	(wire
 		(pts
+			(xy 83.82 24.13) (xy 85.725 24.13)
+		)
+		(stroke
+			(width 0)
+			(type default)
+		)
+	)
+	(wire
+		(pts
 			(xy 247.015 53.34) (xy 247.015 55.88)
 		)
@@
 	(wire
 		(pts
+			(xy 83.82 24.13) (xy 83.82 26.035)
+		)
+		(stroke
+			(width 0)
+			(type default)
+		)
+	)
+	(wire
+		(pts
 			(xy 42.545 41.91) (xy 51.435 41.91)
 		)
@@
 	(wire
 		(pts
-			(xy 93.345 29.21) (xy 93.345 31.75)
+			(xy 93.345 31.75) (xy 93.345 34.29)
 		)
 		(stroke
@@
 	(wire
 		(pts
-			(xy 102.87 21.59) (xy 102.87 23.495)
+			(xy 102.87 21.59) (xy 102.87 26.035)
 		)
 		(stroke
@@
 	(wire
 		(pts
-			(xy 83.82 28.575) (xy 83.82 31.75)
+			(xy 83.82 31.115) (xy 83.82 34.29)
 		)
 		(stroke
@@
 	(wire
 		(pts
-			(xy 83.82 21.59) (xy 83.82 23.495)
+			(xy 83.82 21.59) (xy 83.82 24.13)
 		)
 		(stroke
@@
 	(wire
 		(pts
-			(xy 102.87 28.575) (xy 102.87 31.75)
+			(xy 102.87 31.115) (xy 102.87 34.29)
 		)
 		(stroke
@@
 		)
 	)
+	(label "L_IN"
+		(at 43.815 156.845 180)
+		(fields_autoplaced yes)
+		(effects
+			(font
+				(size 0.7 0.7)
+			)
+			(justify right bottom)
+		)
+	)
 	(label "USB_DPU"
 		(at 212.09 66.04 0)
@@
 		)
 	)
-	(label "USB_DM"
+	(label "USB_DN"
 		(at 212.09 68.58 0)
 		(fields_autoplaced yes)
@@
 		)
 	)
+	(label "L_OUT"
+		(at 53.975 156.845 0)
+		(fields_autoplaced yes)
+		(effects
+			(font
+				(size 0.7 0.7)
+			)
+			(justify left bottom)
+		)
+	)
 	(label "GND"
 		(at 250.825 29.845 0)
@@
 		)
 	)
-	(label "USB_DM"
+	(label "USB_DN"
 		(at 51.435 36.83 180)
 		(fields_autoplaced yes)
@@
 	(symbol
 		(lib_id "Device:C_Small")
-		(at 102.87 26.035 0)
+		(at 102.87 28.575 0)
 		(mirror y)
 		(unit 1)
@@
 		(dnp no)
 		(property "Reference" "C2"
-			(at 104.14 23.495 90)
+			(at 104.14 26.035 90)
 			(effects
 				(font
@@
 		)
 		(property "Value" "10uF"
-			(at 104.14 29.21 90)
+			(at 104.14 31.75 90)
 			(effects
 				(font
@@
 		)
 		(property "Footprint" "Capacitor_SMD:C_0805_2012Metric"
-			(at 102.87 26.035 0)
+			(at 102.87 28.575 0)
 			(effects
 				(font
@@
 		)
 		(property "Datasheet" "~"
-			(at 102.87 26.035 0)
+			(at 102.87 28.575 0)
 			(effects
 				(font
@@
 		)
 		(property "Description" "Unpolarized capacitor, small symbol"
-			(at 102.87 26.035 0)
+			(at 102.87 28.575 0)
 			(effects
 				(font
@@
 	(symbol
 		(lib_id "power:GND")
-		(at 93.345 31.75 0)
+		(at 93.345 34.29 0)
 		(unit 1)
 		(exclude_from_sim no)
@@
 		(dnp no)
 		(property "Reference" "#PWR03"
-			(at 93.345 38.1 0)
+			(at 93.345 40.64 0)
 			(effects
 				(font
@@
 		)
 		(property "Value" "GND"
-			(at 93.345 36.195 0)
+			(at 93.345 38.735 0)
 			(effects
 				(font
@@
 		)
 		(property "Footprint" ""
-			(at 93.345 31.75 0)
+			(at 93.345 34.29 0)
 			(effects
 				(font
@@
 		)
 		(property "Datasheet" ""
-			(at 93.345 31.75 0)
+			(at 93.345 34.29 0)
 			(effects
 				(font
@@
 		)
 		(property "Description" "Power symbol creates a global label with name \"GND\" , ground"
-			(at 93.345 31.75 0)
+			(at 93.345 34.29 0)
 			(effects
 				(font
@@
 	)
 	(symbol
+		(lib_id "Regulator_Linear:AP2112K-3.3")
+		(at 93.345 24.13 0)
+		(unit 1)
+		(exclude_from_sim no)
+		(in_bom yes)
+		(on_board yes)
+		(dnp no)
+		(property "Reference" "U3"
+			(at 88.9 30.48 0)
+			(effects
+				(font
+					(size 1.27 1.27)
+				)
+			)
+		)
+		(property "Value" "AP2112K-3.3"
+			(at 93.345 18.415 0)
+			(effects
+				(font
+					(size 1.27 1.27)
+				)
+			)
+		)
+		(property "Footprint" "Package_TO_SOT_SMD:SOT-23-5"
+			(at 93.345 15.875 0)
+			(effects
+				(font
+					(size 1.27 1.27)
+				)
+				(hide yes)
+			)
+		)
+		(property "Datasheet" "https://www.diodes.com/assets/Datasheets/AP2112.pdf"
+			(at 93.345 21.59 0)
+			(effects
+				(font
+					(size 1.27 1.27)
+				)
+				(hide yes)
+			)
+		)
+		(property "Description" "600mA low dropout linear regulator, with enable pin, 3.8V-6V input voltage range, 3.3V fixed positive output, SOT-23-5"
+			(at 93.345 24.13 0)
+			(effects
+				(font
+					(size 1.27 1.27)
+				)
+				(hide yes)
+			)
+		)
+		(pin "1"
+		)
+		(pin "2"
+		)
+		(pin "5"
+		)
+		(pin "4"
+		)
+		(pin "3"
+		)
+		(instances
+			(project "CCCCPPPS_MkII"
+				(path "/c597219b-55b0-4e5b-b8bf-6d413311061c"
+					(reference "U3")
+					(unit 1)
+				)
+			)
+		)
+	)
+	(symbol
 		(lib_id "Device:R")
 		(at 117.475 184.15 0)
@@
 	(symbol
 		(lib_id "power:GND")
-		(at 83.82 31.75 0)
+		(at 83.82 34.29 0)
 		(unit 1)
 		(exclude_from_sim no)
@@
 		(dnp no)
 		(property "Reference" "#PWR02"
-			(at 83.82 38.1 0)
+			(at 83.82 40.64 0)
 			(effects
 				(font
@@
 		)
 		(property "Value" "GND"
-			(at 83.82 36.195 0)
+			(at 83.82 38.735 0)
 			(effects
 				(font
@@
 		)
 		(property "Footprint" ""
-			(at 83.82 31.75 0)
+			(at 83.82 34.29 0)
 			(effects
 				(font
@@
 		)
 		(property "Datasheet" ""
-			(at 83.82 31.75 0)
+			(at 83.82 34.29 0)
 			(effects
 				(font
@@
 		)
 		(property "Description" "Power symbol creates a global label with name \"GND\" , ground"
-			(at 83.82 31.75 0)
+			(at 83.82 34.29 0)
 			(effects
 				(font
@@
 	(symbol
 		(lib_id "Device:C_Small")
-		(at 83.82 26.035 0)
+		(at 83.82 28.575 0)
 		(unit 1)
 		(exclude_from_sim no)
@@
 		(dnp no)
 		(property "Reference" "C1"
-			(at 82.55 23.495 90)
+			(at 82.55 26.035 90)
 			(effects
 				(font
@@
 		)
 		(property "Value" "10uF"
-			(at 82.55 29.21 90)
+			(at 82.55 31.75 90)
 			(effects
 				(font
@@
 		)
 		(property "Footprint" "Capacitor_SMD:C_0805_2012Metric"
-			(at 83.82 26.035 0)
+			(at 83.82 28.575 0)
 			(effects
 				(font
@@
 		)
 		(property "Datasheet" "~"
-			(at 83.82 26.035 0)
+			(at 83.82 28.575 0)
 			(effects
 				(font
@@
 		)
 		(property "Description" "Unpolarized capacitor, small symbol"
-			(at 83.82 26.035 0)
+			(at 83.82 28.575 0)
 			(effects
 				(font
@@
 	)
 	(symbol
-		(lib_id "Regulator_Linear:AMS1117-3.3")
-		(at 93.345 21.59 0)
-		(unit 1)
-		(exclude_from_sim no)
-		(in_bom yes)
-		(on_board yes)
-		(dnp no)
-		(property "Reference" "U1"
-			(at 89.535 28.575 0)
-			(effects
-				(font
-					(size 1.27 1.27)
-				)
-			)
-		)
-		(property "Value" "AMS1117-3.3"
-			(at 93.345 18.415 0)
-			(effects
-				(font
-					(size 1.27 1.27)
-				)
-			)
-		)
-		(property "Footprint" "Package_TO_SOT_SMD:SOT-223-3_TabPin2"
-			(at 93.345 16.51 0)
-			(effects
-				(font
-					(size 1.27 1.27)
-				)
-				(hide yes)
-			)
-		)
-		(property "Datasheet" "http://www.advanced-monolithic.com/pdf/ds1117.pdf"
-			(at 95.885 27.94 0)
-			(effects
-				(font
-					(size 1.27 1.27)
-				)
-				(hide yes)
-			)
-		)
-		(property "Description" "1A Low Dropout regulator, positive, 3.3V fixed output, SOT-223"
-			(at 93.345 21.59 0)
-			(effects
-				(font
-					(size 1.27 1.27)
-				)
-				(hide yes)
-			)
-		)
-		(pin "1"
-		)
-		(pin "2"
-		)
-		(pin "3"
-		)
-		(instances
-			(project ""
-				(path "/c597219b-55b0-4e5b-b8bf-6d413311061c"
-					(reference "U1")
-					(unit 1)
-				)
-			)
-		)
-	)
-	(symbol
 		(lib_id "Device:R")
 		(at 113.03 184.15 180)
@@
 	(symbol
 		(lib_id "power:GND")
-		(at 102.87 31.75 0)
+		(at 102.87 34.29 0)
 		(unit 1)
 		(exclude_from_sim no)
@@
 		(dnp no)
 		(property "Reference" "#PWR04"
-			(at 102.87 38.1 0)
+			(at 102.87 40.64 0)
 			(effects
 				(font
@@
 		)
 		(property "Value" "GND"
-			(at 102.87 36.195 0)
+			(at 102.87 38.735 0)
 			(effects
 				(font
@@
 		)
 		(property "Footprint" ""
-			(at 102.87 31.75 0)
+			(at 102.87 34.29 0)
 			(effects
 				(font
@@
 		)
 		(property "Datasheet" ""
-			(at 102.87 31.75 0)
+			(at 102.87 34.29 0)
 			(effects
 				(font
@@
 		)
 		(property "Description" "Power symbol creates a global label with name \"GND\" , ground"
-			(at 102.87 31.75 0)
+			(at 102.87 34.29 0)
 			(effects
 				(font

Commit message: Full Refactor
Parts:
- removed C3: 100nF, Capacitor_SMD:C_0805_2012Metric, symbol Device:C_Small
- added JP1: JMP_USB_VIN, Jumper:SolderJumper-2_P1.3mm_Open_RoundedPad1.0x1.5mm, symbol Jumper:Jumper_2_Open
- J1: footprint Connector_PinSocket_2.54mm:PinSocket_1x03_P2.54mm_Vertical -> Connector_PinHeader_2.54mm:PinHeader_1x03_P2.54mm_Vertical
- TP1, TP3, TP4: footprint TestPoint:TestPoint_Pad_D3.0mm -> TestPoint:TestPoint_Pad_D1.5mm
- TP2: value 5V -> VIN; footprint TestPoint:TestPoint_Pad_D3.0mm -> TestPoint:TestPoint_Pad_D1.5mm
Connections:
- net GND: now also J4.1 (Pin_1); no longer J4.2 (Pin_2)
- net VBUS_OUT_NEG: now also J3.1 (Pin_1); no longer J3.2 (Pin_2)
- net VBUS_OUT_POS: now also J3.2 (Pin_2); no longer J3.1 (Pin_1)
- net VBUS_5V_USB renamed VBUS_VIN
- net VBUS_VIN: now also J4.2 (Pin_2), JP1.2 (B); no longer J2.A4 (VBUS), J2.A9 (VBUS), J2.B4 (VBUS), J2.B9 (VBUS), J4.1 (Pin_1)
- new net VBUS_USB: J2.A4 (VBUS), J2.A9 (VBUS), J2.B4 (VBUS), J2.B9 (VBUS), JP1.1 (A)
Other:
- moved on the sheet: C1, C2, J4, U3
